Commit message: implement four thrusters

File: urdf/body.urdf (robot description, URDF)
Before this commit: robot Oke-bot, 3 links, 2 joints
Links:
- removed link thruster_guard_link
- removed link thruster_proppeller_link
- added link thruster_1_guard_link, mass 1.339; collision mesh filename=/home/yasuyuki/vrx_ws/src/vrx/Oke-bot/meshes/STL/thruster_g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 scale=0.001 0.001 0.001; visual mesh filename=/home/yasuyuki/vrx_ws/src/vrx/Oke-bot/meshes/DAE/thruster_g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 scale=0.001 0.001 0.001
- added link thruster_1_propeller_link, mass 0.203; collision mesh filename=/home/yasuyuki/vrx_ws/src/vrx/Oke-bot/meshes/STL/thruster_p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 scale=0.001 0.001 0.001; visual mesh filename=/home/yasuyuki/vrx_ws/src/vrx/Oke-bot/meshes/DAE/thruster_p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 scale=0.001 0.001 0.001
- added link thruster_3_guard_link, mass 1.339; collision mesh filename=/home/yasuyuki/vrx_ws/src/vrx/Oke-bot/meshes/STL/thruster_g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 scale=0.001 0.001 0.001; visual mesh filename=/home/yasuyuki/vrx_ws/src/vrx/Oke-bot/meshes/DAE/thruster_g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 scale=0.001 0.001 0.001
- link okebot_base_link: geometry collision mesh filename=/home/yasuyuki/vrx_ws/src/vrx/Oke-bot/meshes/STL/okebot_fra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 scale=0.001 0.001 0.001; visual mesh filename=/home/yasuyuki/vrx_ws/src/vrx/Oke-bot/meshes/DAE/Okebot_fra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 scale=0.001 0.001 0.001
Joints:
- removed joint frame_guard_joint
- removed joint guard_propeller_joint
- added joint thruster_1_joint: type continuous, parent thruster_1_guard_link, child thruster_1_propeller_link, origin xyz=0 0 0 rpy=0 0 0, axis 0 1 0
- added joint thruster_3_joint: type fixed, parent okebot_base_link, child thruster_3_guard_link, origin xyz=0.115 -0.007 -0.099 rpy=0 0 3.141592

File: urdf/body.urdf.xacro (robot description, xacro)
@@ -1,2 +1,204 @@
+<?xml version="1.0"?>
+<robot xmlns:xacro="http://www.ros.org/wiki/xacro" name="Oke-bot" >
+  	<xacro:include filename="$(find Oke-bot)/urdf/materials.urdf.xacro" />
+	<xacro:property name="body_file" value="$(find Oke-bot)/meshes/DAE/Okebot_framev2.dae"/>
+	<xacro:property name="guard_file" value="$(find Oke-bot)/meshes/DAE/thruster_guardv2.dae"/>
+	<xacro:property name="propeller_file" value="$(find Oke-bot)/meshes/DAE/thruster_propeller.dae"/>
+	<xacro:property name="body_collision" value="$(find Oke-bot)/meshes/STL/okebot_framev2.stl"/>
+	<xacro:property name="guard_collision" value="$(find Oke-bot)/meshes/STL/thruster_guard.stl"/>
+	<xacro:property name="propeller_collision" value="$(find Oke-bot)/meshes/STL/thruster_propeller.stl"/>
+	<xacro:property name="frame_mass" value="5.0"/>
+	<xacro:property name="guard_mass" value="1.339"/>
+	<xacro:property name="propeller_mass" value="0.203"/>
+	<xacro:property name="guard_length_x1" value="0.115"/>
+	<xacro:property name="guard_length_x2" value="0.005"/>
+	<xacro:property name="guard_length_y1" value="-0.007"/>
+	<xacro:property name="guard_length_y2" value="0.115"/>
+	<xacro:property name="guard_length_y3" value="0.005."/>
+	<xacro:property name="guard_height" value="-0.099"/>
+	<xacro:property name="PI" value="3.141592"/>
+	<link name="okebot_base_link">
+	  	<inertial>
+	    	<mass value="${frame_mass}"/>
+	      	<inertia ixx = "1.988E+08"  ixy ="-1.016E+05"  ixz = "6.901E+06"
+					 iyx = "-1.016E+05" iyy = "3.364E+08"  iyz = "-8.738E+04"
+					 izx = "6.901E+06"  izy = "-8.738E+04"  izz = "1.988E+08"/>
+	    </inertial>
+	    <visual>
+			<origin xyz="0 0 0" rpy="0 0 0"/>
+	      	<geometry>
+	      		<mesh filename="${body_file}" scale="0.001 0.001 0.001"/>
+	      	</geometry>
+	    </visual>
+	    <collision>
+	      	<geometry>
+	      		<mesh filename="${body_collision}" scale="0.001 0.001 0.001"/>
+	        </geometry>
+	  	</collision>
+	</link>
+	<xacro:macro name="guard_template" params="name length_x length_y yaw">
+		<joint name="${name}_joint" type="fixed">
+			<parent link="okebot_base_link"/>
+			<child link="${name}_guard_link"/>
+			<origin xyz="${length_x} ${length_y} ${guard_height}" rpy="0 0 ${yaw}"/>
+		</joint>
+		<link name="${name}_guard_link">
+			<inertial>
+				<mass value="${guard_mass}"/>
+		      	<inertia ixx = "1.227E+06"  ixy = "22.808"     ixz = "12.874"
+						 iyx = "22.808"     iyy = "1.189E+06"  iyz = "7036.714"
+						 izx = "12.874"     izy = "7036.714"   izz = "1.374E+06"/>
+			</inertial>
+		    <visual>
+		      	<geometry>
+		      		<mesh filename="${guard_file}" scale="0.001 0.001 0.001"/>
+		      	</geometry>
+		    </visual>
+		    <collision>
+				<origin xyz="${length_x} ${length_y} ${guard_height}" rpy="0 0 ${yaw}"/>
+		      	<geometry>
+		      		<mesh filename="${guard_collision}" scale="0.001 0.001 0.001"/>
+		        </geometry>
+		  	</collision>
+		</link>
+	</xacro:macro>
+	<!--
+	<xacro:macro name="propeller_template" params="name length_x length_y yaw">
+		<joint name="${name}_joint" type="continuous">
+			<parent link="${name}_guard_link"/>
+			<child link="${name}_propeller_link"/>
+			<axis xyz="0 1 0"/>
+			<origin xyz="0 0 0" rpy="0 0 0"/>
+		</joint>
+		<link name="${name}_propeller_link">
+			<inertial>
+				<mass value="${propeller_mass}"/>
+		      	<inertia ixx = "2.964E+04"  ixy = "1652.571"  ixz = "-2.620E-08"
+						 iyx = "1652.571"   iyy = "2.746E+04" iyz = "2.516E-07"
+						 izx = "-2.620E-08" izy = "2.516E-07" izz = "4.384E+04"/>
+			</inertial>
+		    <visual>
+		      	<geometry>
+		      		<mesh filename="${propeller_file}" scale="0.001 0.001 0.001"/>
+		      	</geometry>
+		    </visual>
+		    <collision>
+				<origin xyz="${length_x} ${length_y} ${guard_height}" rpy="0 0 ${yaw}"/>
+		      	<geometry>
+		      		<mesh filename="${propeller_collision}" scale="0.001 0.001 0.001"/>
+		        </geometry>
+		  	</collision>
+		</link>
+	</xacro:macro>
+	-->
+	<xacro:guard_template name="thruster_1" length_x="${-guard_length_x1}" length_y="${guard_length_y1}" yaw="0"/>
+	<xacro:guard_template name="thruster_2" length_x="${guard_length_x2}" length_y="${guard_length_y2}" yaw="${PI/2}"/>
+	<xacro:guard_template name="thruster_3" length_x="${guard_length_x1}" length_y="${guard_length_y1}" yaw="${PI}"/>
+	<xacro:guard_template name="thruster_4" length_x="${guard_length_x2}" length_y="${-guard_length_y2}" yaw="${-PI/2}"/>
+	<!--
+	<xacro:propeller_template name="thruster_1" length_x="${-guard_length_x1}" length_y="${guard_length_y1}" yaw="0"/>
+	-->
+	<joint name="propeller_1_joint" type="continuous">
+		<origin xyz="0 0 0" rpy="0 0 0"/>
+		<axis xyz="0 1 0"/>
+		<parent link="thruster_1_guard_link"/>
+		<child link="propeller_1_link"/>
+	</joint>
+	<link name="propeller_1_link">
+		<inertial>
+			<mass value="${propeller_mass}"/>
+	      	<inertia ixx = "2.964E+04"  ixy = "1652.571"  ixz = "-2.620E-08"
+					 iyx = "1652.571"   iyy = "2.746E+04" iyz = "2.516E-07"
+					 izx = "-2.620E-08" izy = "2.516E-07" izz = "4.384E+04"/>
+		</inertial>
+	    <visual>
+	      	<geometry>
+	      		<mesh filename="${propeller_file}" scale="0.001 0.001 0.001"/>
+	      	</geometry>
+	    </visual>
+	    <collision>
+			<origin xyz="${-guard_length_x1} ${guard_length_y1} ${guard_height}" rpy="0 0 0"/>
+	      	<geometry>
+	      		<mesh filename="${propeller_collision}" scale="0.001 0.001 0.001"/>
+	        </geometry>
+	  	</collision>
+	</link>
+	<joint name="propeller_2_joint" type="continuous">
+		<origin xyz="0 0 0" rpy="0 0 0"/>
+		<axis xyz="0 1 0"/>
+		<parent link="thruster_2_guard_link"/>
+		<child link="propeller_2_link"/>
+	</joint>
+	<link name="propeller_2_link">
+		<inertial>
+			<mass value="${propeller_mass}"/>
+	      	<inertia ixx = "2.964E+04"  ixy = "1652.571"  ixz = "-2.620E-08"
+					 iyx = "1652.571"   iyy = "2.746E+04" iyz = "2.516E-07"
+					 izx = "-2.620E-08" izy = "2.516E-07" izz = "4.384E+04"/>
+		</inertial>
+	    <visual>
+	      	<geometry>
+	      		<mesh filename="${propeller_file}" scale="0.001 0.001 0.001"/>
+	      	</geometry>
+	    </visual>
+	    <collision>
+			<origin xyz="${guard_length_x2} ${guard_length_y2} ${guard_height}" rpy="0 0 0"/>
+	      	<geometry>
+	      		<mesh filename="${propeller_collision}" scale="0.001 0.001 0.001"/>
+	        </geometry>
+	  	</collision>
+	</link>
+	<joint name="propeller_3_joint" type="continuous">
+		<origin xyz="0 0 0" rpy="0 0 0"/>
+		<axis xyz="0 1 0"/>
+		<parent link="thruster_3_guard_link"/>
+		<child link="propeller_3_link"/>
+	</joint>
+	<link name="propeller_3_link">
+		<inertial>
+			<mass value="${propeller_mass}"/>
+	      	<inertia ixx = "2.964E+04"  ixy = "1652.571"  ixz = "-2.620E-08"
+					 iyx = "1652.571"   iyy = "2.746E+04" iyz = "2.516E-07"
+					 izx = "-2.620E-08" izy = "2.516E-07" izz = "4.384E+04"/>
+		</inertial>
+	    <visual>
+	      	<geometry>
+	      		<mesh filename="${propeller_file}" scale="0.001 0.001 0.001"/>
+	      	</geometry>
+	    </visual>
+	    <collision>
+			<origin xyz="${guard_length_x1} ${guard_length_y1} ${guard_height}" rpy="0 0 0"/>
+	      	<geometry>
+	      		<mesh filename="${propeller_collision}" scale="0.001 0.001 0.001"/>
+	        </geometry>
+	  	</collision>
+	</link>
+	<joint name="propeller_4_joint" type="continuous">
+		<origin xyz="0 0 0" rpy="0 0 0"/>
+		<axis xyz="0 1 0"/>
+		<parent link="thruster_4_guard_link"/>
+		<child link="propeller_4_link"/>
+	</joint>
+	<link name="propeller_4_link">
+		<inertial>
+			<mass value="${propeller_mass}"/>
+	      	<inertia ixx = "2.964E+04"  ixy = "1652.571"  ixz = "-2.620E-08"
+					 iyx = "1652.571"   iyy = "2.746E+04" iyz = "2.516E-07"
+					 izx = "-2.620E-08" izy = "2.516E-07" izz = "4.384E+04"/>
+		</inertial>
+	    <visual>
+	      	<geometry>
+	      		<mesh filename="${propeller_file}" scale="0.001 0.001 0.001"/>
+	      	</geometry>
+	    </visual>
+	    <collision>
+			<origin xyz="${guard_length_x2} ${-guard_length_y2} ${guard_height}" rpy="0 0 0"/>
+	      	<geometry>
+	      		<mesh filename="${propeller_collision}" scale="0.001 0.001 0.001"/>
+	        </geometry>
+	  	</collision>
+	</link>
+</robot>
+<!--
 <?xml version="1.0"?>
 <robot xmlns:xacro="http://www.ros.org/wiki/xacro" name="Oke-bot" >
@@ -62,6 +264,7 @@
 	  	</collision>
 	</link>
-	<joint name="guard_propeller_joint" type="fixed">
-		<origin xyz="0 0 0" rpy="0 0 0"/>
+	<joint name="guard_propeller_joint" type="continuous">
+		<origin xyz="0 0 0" rpy="0 0 0"/>
+		<axis xyz="0 1 0"/>
 		<parent link="thruster_guard_link"/>
 		<child link="thruster_propeller_link"/>
@@ -87,2 +290,3 @@
 	</link>
 </robot>
+-->
