Commit message: assemble thruster to base

File: urdf/body.urdf.xacro (robot description, xacro)
@@ -1,21 +1,20 @@
 <?xml version="1.0"?>
 <robot xmlns:xacro="http://www.ros.org/wiki/xacro" name="Oke-bot" >
-	<xacro:property name="Oke-bot_frame_file" value="package://Oke-bot/meshes/Okebot_framedae"/>
-	<xacro:property name="thruster_guard_file" value="package://Oke-bot/meshes/thruster_guard.dae"/>
-	<xacro:property name="thruster_propeller_file" value="package://Oke-bot/meshes/thruster_proppeller.dae"/>
+	<xacro:property name="body_file" value="$(find Oke-bot)/meshes/DAE/Okebot_framev2.dae"/>
+	<xacro:property name="thruster_guard_file" value="$(find Oke-bot)/meshes/DAE/thruster_guardv2.dae"/>
+	<xacro:property name="thruster_propeller_file" value="$(find Oke-bot)/meshes/DAE/thruster_propeller.dae"/>
+	<xacro:property name="body_collision" value="$(find Oke-bot)/meshes/STL/okebot_framev2.stl"/>
+	<xacro:property name="thruster_guard_collision" value="$(find Oke-bot)/meshes/STL/thruster_guard.stl"/>
+	<xacro:property name="thruster_propeller_collision" value="$(find Oke-bot)/meshes/STL/thruster_propeller.stl"/>
 	<xacro:property name="frame_mass" value="5.0"/>
-	<xacro:property name="gurad_mass" value="1.339"/>
+	<xacro:property name="guard_mass" value="1.339"/>
 	<xacro:property name="propeller_mass" value="0.203"/>
 	<xacro:property name="guard_length_x1" value="0.115"/>
 	<xacro:property name="guard_length_x2" value="0.005"/>
-	<xacro:property name="guard_length_z1" value="-0.007"/>
-	<xacro:property name="guard_length_z2" value="0.115"/>
-	<xacro:property name="guard_length_z3" value="0.005."/>
+	<xacro:property name="guard_length_y1" value="-0.007"/>
+	<xacro:property name="guard_length_y2" value="0.115"/>
+	<xacro:property name="guard_length_y3" value="0.005."/>
 	<xacro:property name="guard_height" value="-0.099"/>
-	<xacro:property name="propeller_length_x" value=""/>
-	<xacro:property name="propeller_length_y" value=""/>
-	<xacro:property name="propeller_length_z" value=""/>
 	<link name="okebot_base_link">
-		<!-- inertial(material, iner)-->
 	  	<inertial>
 	    	<mass value="${frame_mass}"/>
@@ -25,14 +24,23 @@
 	    	</inertial>
 	    <visual>
+			<origin xyz="0 0 0" rpy="0 0 0"/>
 	      	<geometry>
-	      		<mesh filename="${visual_mesh_file}" scale="0.001 0.001 0.001"/>
+	      		<mesh filename="${body_file}" scale="0.001 0.001 0.001"/>
 	      	</geometry>
+	      <material name="black">
+			<color rgba="0 0 0 1" />
+		  </material>
 	    </visual>
 	    <collision>
 	      	<geometry>
-	          <box size="0.384 0.300 0.384"/>
+	      		<mesh filename="${body_collision}" scale="0.001 0.001 0.001"/>
 	        </geometry>
 	  	</collision>
 	</link>
+	<joint name="frame_guard_joint" type="fixed">
+		<origin xyz="${guard_length_x1} ${guard_length_y1} ${guard_height}" rpy="0 0 0"/>
+		<parent link="okebot_base_link"/>
+		<child link="thruster_guard_link"/>
+	</joint>
 	<link name="thruster_guard_link">
 		<inertial>
@@ -41,5 +49,4 @@
 					 iyx = "22.808"     iyy = "1.189E+06"  iyz = "7036.714"
 					 izx = "12.874"     izy = "7036.714"   izz = "1.374E+06"/>
-	    	</inertial>
 		</inertial>
 	    <visual>
@@ -48,6 +55,17 @@
 	      	</geometry>
 	    </visual>
+	    <collision>
+			<origin xyz="${guard_length_x1} ${guard_length_y1} ${guard_height}" rpy="0 0 0"/>
+	      	<geometry>
+	      		<mesh filename="${thruster_guard_collision}" scale="0.001 0.001 0.001"/>
+	        </geometry>
+	  	</collision>
 	</link>
-	<link name="thruster_proppeller_link">
+	<joint name="guard_propeller_joint" type="fixed">
+		<origin xyz="0 0 0" rpy="0 0 0"/>
+		<parent link="thruster_guard_link"/>
+		<child link="thruster_propeller_link"/>
+	</joint>
+	<link name="thruster_propeller_link">
 		<inertial>
 			<mass value="${propeller_mass}"/>
@@ -55,5 +73,4 @@
 					 iyx = "1652.571"   iyy = "2.746E+04" iyz = "2.516E-07"
 					 izx = "-2.620E-08" izy = "2.516E-07" izz = "4.384E+04"/>
-	    	</inertial>
 		</inertial>
 	    <visual>
@@ -62,14 +79,10 @@
 	      	</geometry>
 	    </visual>
+	    <collision>
+			<origin xyz="${guard_length_x1} ${guard_length_y1} ${guard_height}" rpy="0 0 0"/>
+	      	<geometry>
+	      		<mesh filename="${thruster_propeller_collision}" scale="0.001 0.001 0.001"/>
+	        </geometry>
+	  	</collision>
 	</link>
-	<joint name="frame_guard_joint">
-		<origin xyz="${guard_length_x1} ${guard_height} ${guard_length_z1}" rpy="0 0 180"/>
-		<parent link="okebot_base_link"/>
-		<child link="thruster_guard_link"/>
-	</joint>
-	<joint name="guard_propeller_joint">
-		<origin xyz="${guard_length_x1} ${guard_height} ${guard_length_z1}" rpy="0 0 180"/>
-		<parent link="thruster_guard_link"/>
-		<child link="thruster_propeller_link"/>
-	</joint>
 </robot>

Commit message: fix xacro file

File: urdf/body.urdf.xacro (robot description, xacro)
@@ -200,93 +200,2 @@
 	</link>
 </robot>
-<!--
-<?xml version="1.0"?>
-<robot xmlns:xacro="http://www.ros.org/wiki/xacro" name="Oke-bot" >
-	<xacro:property name="body_file" value="$(find Oke-bot)/meshes/DAE/Okebot_framev2.dae"/>
-	<xacro:property name="thruster_guard_file" value="$(find Oke-bot)/meshes/DAE/thruster_guardv2.dae"/>
-	<xacro:property name="thruster_propeller_file" value="$(find Oke-bot)/meshes/DAE/thruster_propeller.dae"/>
-	<xacro:property name="body_collision" value="$(find Oke-bot)/meshes/STL/okebot_framev2.stl"/>
-	<xacro:property name="thruster_guard_collision" value="$(find Oke-bot)/meshes/STL/thruster_guard.stl"/>
-	<xacro:property name="thruster_propeller_collision" value="$(find Oke-bot)/meshes/STL/thruster_propeller.stl"/>
-	<xacro:property name="frame_mass" value="5.0"/>
-	<xacro:property name="guard_mass" value="1.339"/>
-	<xacro:property name="propeller_mass" value="0.203"/>
-	<xacro:property name="guard_length_x1" value="0.115"/>
-	<xacro:property name="guard_length_x2" value="0.005"/>
-	<xacro:property name="guard_length_y1" value="-0.007"/>
-	<xacro:property name="guard_length_y2" value="0.115"/>
-	<xacro:property name="guard_length_y3" value="0.005."/>
-	<xacro:property name="guard_height" value="-0.099"/>
-	<link name="okebot_base_link">
-	  	<inertial>
-	    	<mass value="${frame_mass}"/>
-	      	<inertia ixx = "1.988E+08"  ixy ="-1.016E+05"  ixz = "6.901E+06"
-					 iyx = "-1.016E+05" iyy = "3.364E+08"  iyz = "-8.738E+04"
-					 izx = "6.901E+06"  izy = "-8.738E+04"  izz = "1.988E+08"/>
-	    	</inertial>
-	    <visual>
-			<origin xyz="0 0 0" rpy="0 0 0"/>
-	      	<geometry>
-	      		<mesh filename="${body_file}" scale="0.001 0.001 0.001"/>
-	      	</geometry>
-	      <material name="black">
-			<color rgba="0 0 0 1" />
-		  </material>
-	    </visual>
-	    <collision>
-	      	<geometry>
-	      		<mesh filename="${body_collision}" scale="0.001 0.001 0.001"/>
-	        </geometry>
-	  	</collision>
-	</link>
-	<joint name="frame_guard_joint" type="fixed">
-		<origin xyz="${guard_length_x1} ${guard_length_y1} ${guard_height}" rpy="0 0 0"/>
-		<parent link="okebot_base_link"/>
-		<child link="thruster_guard_link"/>
-	</joint>
-	<link name="thruster_guard_link">
-		<inertial>
-			<mass value="${guard_mass}"/>
-	      	<inertia ixx = "1.227E+06"  ixy = "22.808"     ixz = "12.874"
-					 iyx = "22.808"     iyy = "1.189E+06"  iyz = "7036.714"
-					 izx = "12.874"     izy = "7036.714"   izz = "1.374E+06"/>
-		</inertial>
-	    <visual>
-	      	<geometry>
-	      		<mesh filename="${thruster_guard_file}" scale="0.001 0.001 0.001"/>
-	      	</geometry>
-	    </visual>
-	    <collision>
-			<origin xyz="${guard_length_x1} ${guard_length_y1} ${guard_height}" rpy="0 0 0"/>
-	      	<geometry>
-	      		<mesh filename="${thruster_guard_collision}" scale="0.001 0.001 0.001"/>
-	        </geometry>
-	  	</collision>
-	</link>
-	<joint name="guard_propeller_joint" type="continuous">
-		<origin xyz="0 0 0" rpy="0 0 0"/>
-		<axis xyz="0 1 0"/>
-		<parent link="thruster_guard_link"/>
-		<child link="thruster_propeller_link"/>
-	</joint>
-	<link name="thruster_propeller_link">
-		<inertial>
-			<mass value="${propeller_mass}"/>
-	      	<inertia ixx = "2.964E+04"  ixy = "1652.571"  ixz = "-2.620E-08"
-					 iyx = "1652.571"   iyy = "2.746E+04" iyz = "2.516E-07"
-					 izx = "-2.620E-08" izy = "2.516E-07" izz = "4.384E+04"/>
-		</inertial>
-	    <visual>
-	      	<geometry>
-	      		<mesh filename="${thruster_propeller_file}" scale="0.001 0.001 0.001"/>
-	      	</geometry>
-	    </visual>
-	    <collision>
-			<origin xyz="${guard_length_x1} ${guard_length_y1} ${guard_height}" rpy="0 0 0"/>
-	      	<geometry>
-	      		<mesh filename="${thruster_propeller_collision}" scale="0.001 0.001 0.001"/>
-	        </geometry>
-	  	</collision>
-	</link>
-</robot>
--->

Commit message: add options

File: urdf/body.urdf.xacro (robot description, xacro)
@@ -5,5 +5,5 @@
 	<xacro:property name="guard_file" value="$(find Oke-bot)/meshes/DAE/thruster_guardv2.dae"/>
 	<xacro:property name="propeller_file" value="$(find Oke-bot)/meshes/DAE/thruster_propeller.dae"/>
-	<xacro:property name="body_collision" value="$(find Oke-bot)/meshes/STL/okebot_framev2.stl"/>
+	<xacro:property name="body_collision" value="$(find Oke-bot)/meshes/STL/Oke-bot_v12.stl"/>
 	<xacro:property name="guard_collision" value="$(find Oke-bot)/meshes/STL/thruster_guard.stl"/>
 	<xacro:property name="propeller_collision" value="$(find Oke-bot)/meshes/STL/thruster_propeller.stl"/>
@@ -55,10 +55,4 @@
 		      	</geometry>
 		    </visual>
-		    <collision>
-				<origin xyz="${length_x} ${length_y} ${guard_height}" rpy="0 0 ${yaw}"/>
-		      	<geometry>
-		      		<mesh filename="${guard_collision}" scale="0.001 0.001 0.001"/>
-		        </geometry>
-		  	</collision>
 		</link>
 	</xacro:macro>
@@ -112,15 +106,4 @@
 					 izx = "-2.620E-08" izy = "2.516E-07" izz = "4.384E+04"/>
 		</inertial>
-	    <visual>
-	      	<geometry>
-	      		<mesh filename="${propeller_file}" scale="0.001 0.001 0.001"/>
-	      	</geometry>
-	    </visual>
-	    <collision>
-			<origin xyz="${-guard_length_x1} ${guard_length_y1} ${guard_height}" rpy="0 0 0"/>
-	      	<geometry>
-	      		<mesh filename="${propeller_collision}" scale="0.001 0.001 0.001"/>
-	        </geometry>
-	  	</collision>
 	</link>
 	<joint name="propeller_2_joint" type="continuous">
@@ -142,10 +125,4 @@
 	      	</geometry>
 	    </visual>
-	    <collision>
-			<origin xyz="${guard_length_x2} ${guard_length_y2} ${guard_height}" rpy="0 0 0"/>
-	      	<geometry>
-	      		<mesh filename="${propeller_collision}" scale="0.001 0.001 0.001"/>
-	        </geometry>
-	  	</collision>
 	</link>
 	<joint name="propeller_3_joint" type="continuous">
@@ -162,15 +139,4 @@
 					 izx = "-2.620E-08" izy = "2.516E-07" izz = "4.384E+04"/>
 		</inertial>
-	    <visual>
-	      	<geometry>
-	      		<mesh filename="${propeller_file}" scale="0.001 0.001 0.001"/>
-	      	</geometry>
-	    </visual>
-	    <collision>
-			<origin xyz="${guard_length_x1} ${guard_length_y1} ${guard_height}" rpy="0 0 0"/>
-	      	<geometry>
-	      		<mesh filename="${propeller_collision}" scale="0.001 0.001 0.001"/>
-	        </geometry>
-	  	</collision>
 	</link>
 	<joint name="propeller_4_joint" type="continuous">
@@ -192,10 +158,4 @@
 	      	</geometry>
 	    </visual>
-	    <collision>
-			<origin xyz="${guard_length_x2} ${-guard_length_y2} ${guard_height}" rpy="0 0 0"/>
-	      	<geometry>
-	      		<mesh filename="${propeller_collision}" scale="0.001 0.001 0.001"/>
-	        </geometry>
-	  	</collision>
 	</link>
 </robot>
